File: SwarmBotTop/Programmer.sch (KiCad schematic (older format))
At the start: 11 parts, among them J4 USB_B_Micro, Q1 MMBT3904, Q2 MMBT3904, U1 CP2102N-A01-GQFN24, U2 MIC5366-3.3YC5

Commit message: Camera routing with all sensors and motors
Parts:
- removed Q1, Q2: MMBT3904, Package_TO_SOT_SMD:SOT-23, symbol Transistor_BJT:MMBT3904
- added Q1: MBT3904DW1, Package_TO_SOT_SMD:SOT-363_SC-70-6, symbol Transistor_BJT:MBT3904DW1
- C5: value C -> 4.7uF
- C6: value C -> 0.1uF
- C7, C8: value C -> 1uF
- R3, R4: value R -> 10K
Changed lines of the file:
@@
 AR Path="/5DAF9EB1/5DE5FC55/5DE5FE02" Ref="C5"  Part="1"
 F 0 "C5" H 5665 2096 50  0000 L CNN
-F 1 "C" H 5665 2005 50  0000 L CNN
+F 1 "4.7uF" H 5665 2005 50  0000 L CNN
 F 2 "Capacitor_SMD:C_0402_1005Metric" H 5588 1900 50  0001 C CNN
 F 3 "~" H 5550 2050 50  0001 C CNN
@@
 AR Path="/5DAF9EB1/5DE5FC55/5DE5FE09" Ref="C6"  Part="1"
 F 0 "C6" H 6015 2096 50  0000 L CNN
-F 1 "C" H 6015 2005 50  0000 L CNN
+F 1 "0.1uF" H 6015 2005 50  0000 L CNN
 F 2 "Capacitor_SMD:C_0402_1005Metric" H 5938 1900 50  0001 C CNN
 F 3 "~" H 5900 2050 50  0001 C CNN
@@
 NoConn ~ 4900 2900
 NoConn ~ 4900 3000
-$Comp
-L Transistor_BJT:MMBT3904 Q?
-U 1 1 5DE645B5
-P 8050 5200
-AR Path="/5DAF9EB1/5DE645B5" Ref="Q?"  Part="1"
-AR Path="/5DAF9EB1/5DE5FC55/5DE645B5" Ref="Q2"  Part="1"
-F 0 "Q2" V 8285 5200 50  0000 C CNN
-F 1 "MMBT3904" V 8376 5200 50  0000 C CNN
-F 2 "Package_TO_SOT_SMD:SOT-23" H 8250 5125 50  0001 L CIN
-F 3 "https://www.fairchildsemi.com/datasheets/2N/2N3904.pdf" H 8050 5200 50  0001 L CNN
-	1    8050 5200
-	0    1    1    0
-$EndComp
-$Comp
-L Transistor_BJT:MMBT3904 Q?
-U 1 1 5DE645BC
-P 7300 5200
-AR Path="/5DAF9EB1/5DE645BC" Ref="Q?"  Part="1"
-AR Path="/5DAF9EB1/5DE5FC55/5DE645BC" Ref="Q1"  Part="1"
-F 0 "Q1" V 7535 5200 50  0000 C CNN
-F 1 "MMBT3904" V 7626 5200 50  0000 C CNN
-F 2 "Package_TO_SOT_SMD:SOT-23" H 7500 5125 50  0001 L CIN
-F 3 "https://www.fairchildsemi.com/datasheets/2N/2N3904.pdf" H 7300 5200 50  0001 L CNN
-	1    7300 5200
-	0    -1   1    0
-$EndComp
 Text Label 7500 5300 0    50   ~ 0
 DTR
@@
 AR Path="/5DAF9EB1/5DE5FC55/5DE645C5" Ref="R3"  Part="1"
 F 0 "R3" H 7370 4896 50  0000 L CNN
-F 1 "R" H 7370 4805 50  0000 L CNN
+F 1 "10K" H 7370 4805 50  0000 L CNN
 F 2 "Resistor_SMD:R_0402_1005Metric" V 7230 4850 50  0001 C CNN
 F 3 "~" H 7300 4850 50  0001 C CNN
@@
 AR Path="/5DAF9EB1/5DE5FC55/5DE645CD" Ref="R4"  Part="1"
 F 0 "R4" H 8120 4896 50  0000 L CNN
-F 1 "R" H 8120 4805 50  0000 L CNN
+F 1 "10K" H 8120 4805 50  0000 L CNN
 F 2 "Resistor_SMD:R_0402_1005Metric" V 7980 4850 50  0001 C CNN
 F 3 "~" H 8050 4850 50  0001 C CNN
@@
 AR Path="/5DAF9EB1/5DE5FC55/5DE67C40" Ref="C8"  Part="1"
 F 0 "C8" H 9315 2746 50  0000 L CNN
-F 1 "C" H 9315 2655 50  0000 L CNN
+F 1 "1uF" H 9315 2655 50  0000 L CNN
 F 2 "Capacitor_SMD:C_0402_1005Metric" H 9238 2550 50  0001 C CNN
 F 3 "~" H 9200 2700 50  0001 C CNN
@@
 AR Path="/5DAF9EB1/5DE5FC55/5DE67C47" Ref="C7"  Part="1"
 F 0 "C7" H 8015 2746 50  0000 L CNN
-F 1 "C" H 8015 2655 50  0000 L CNN
+F 1 "1uF" H 8015 2655 50  0000 L CNN
 F 2 "Capacitor_SMD:C_0402_1005Metric" H 7938 2550 50  0001 C CNN
 F 3 "~" H 7900 2700 50  0001 C CNN
@@
 	0    -1   -1   0
 $EndComp
+$Comp
+L Transistor_BJT:MBT3904DW1 Q1
+U 1 1 5DF31040
+P 8050 5200
+F 0 "Q1" V 8285 5200 50  0000 C CNN
+F 1 "MBT3904DW1" V 8376 5200 50  0000 C CNN
+F 2 "Package_TO_SOT_SMD:SOT-363_SC-70-6" H 8250 5300 50  0001 C CNN
+F 3 "http://www.onsemi.com/pub_link/Collateral/MBT3904DW1T1-D.PDF" H 8050 5200 50  0001 C CNN
+	1    8050 5200
+	0    1    1    0
+$EndComp
+$Comp
+L Transistor_BJT:MBT3904DW1 Q1
+U 2 1 5DF348BB
+P 7300 5200
+F 0 "Q1" V 7535 5200 50  0000 C CNN
+F 1 "MBT3904DW1" V 7626 5200 50  0000 C CNN
+F 2 "Package_TO_SOT_SMD:SOT-363_SC-70-6" H 7500 5300 50  0001 C CNN
+F 3 "http://www.onsemi.com/pub_link/Collateral/MBT3904DW1T1-D.PDF" H 7300 5200 50  0001 C CNN
+	2    7300 5200
+	0    -1   1    0
+$EndComp
 $EndSCHEMATC
